File: KunaiGC_main/KunaiGC_main.kicad_sch (KiCad schematic)
At the start: 18 parts, among them J1 Conn_01x06, J2 Conn_01x01, J3 Conn_02x04_Counter_Clockwise, J4 Conn_02x04_Counter_Clockwise, J5 Conn_01x06, U1 XC9536VQ44, U2 M25P40

Commit message: updated to latest files
Connections:
- net EXI.CLK: now also U1.44 (I/O/GCK2)
